Commit message: Added imu sensor and adjusted parameters

File: urdf/swd_starter_kit_with_ex_tool.urdf (robot description, URDF)
Before this commit: robot swd_starter_kit, 8 links, 7 joints
Links:
- removed link base_footprint
- removed link imu_link
- added link imu_sensor_link, mass 0.1; collision box size=0.055 0.0368 0.024
Joints:
- removed joint base_joint
- joint base_imu_link: child imu_link -> imu_sensor_link
